Commit message: moved files into more appropriate folders

File: models/so100.urdf (robot description, URDF)
Before this commit: robot so_arm100, 7 links, 6 joints
Links:
- link base: geometry collision mesh filename=../assets/Base.stl; visual mesh filename=../assets/Base.stl
- link gripper: geometry visual mesh filename=../assets/Fixed_Jaw.stl; visual mesh filename=../assets/Fixed_Jaw_Motor.stl
- link jaw: geometry visual mesh filename=../assets/Moving_Jaw.stl
- link lower_arm: geometry collision mesh filename=../assets/Lower_Arm.stl; visual mesh filename=../assets/Lower_Arm.stl
- link shoulder: geometry collision mesh filename=../assets/Rotation_Pitch.stl; visual mesh filename=../assets/Rotation_Pitch.stl
- link upper_arm: geometry collision mesh filename=../assets/Upper_Arm.stl; visual mesh filename=../assets/Upper_Arm.stl
- link wrist: geometry collision mesh filename=../assets/Wrist_Pitch_Roll.stl; visual mesh filename=../assets/Wrist_Pitch_Roll.stl
